File: hardware/quadrature_generator.sch (EAGLE design)
At the start: 38 parts, among them IC1 74LVC1G14, IC2 74LVC74, IC3 74LVC04, IC4 74LVC04, IC5 PT7C4511, IC6 78L33

Commit message: checkpoint
Parts:
- C1, C10, C11, C2, C3, C4, C5, C6, C7, C8, C9: device vna_adapter:C0805 -> quadrature_generator:C0805
- IC1: device vna_adapter:74LVC1G14 -> quadrature_generator:74LVC1G14
- IC2: device vna_adapter:74LVC74 -> quadrature_generator:74LVC74
- IC3, IC4: device vna_adapter:74LVC04 -> quadrature_generator:74LVC04
- IC5: device vna_adapter:PT7C4511 -> quadrature_generator:PT7C4511
- IC6: device vna_adapter:REGULATOR_3TERM -> quadrature_generator:REGULATOR_3TERM
- J_F_IN, J_IN_PHASE, J_QUADRATURE: device vna_adapter:EDGE_LAUNCH_JACK -> quadrature_generator:EDGE_LAUNCH_JACK
- R1, R4, R5: device vna_adapter:R1206 -> quadrature_generator:R1206
- R2, R3: device vna_adapter:R0805 -> quadrature_generator:R0805
- U$1: device vna_adapter:FT37_TRIFILAR_1 -> quadrature_generator:FT37_TRIFILAR_1
- U$18: device vna_adapter:USB_JACK -> quadrature_generator:USB_JACK
- U$26, U$32, U$33, U$34, U$35, U$36, U$37, U$42, U$43: device vna_adapter:SOLDER_BRIDGE -> quadrature_generator:SOLDER_BRIDGE
- U$50: device vna_adapter:MMBD7000L -> quadrature_generator:MMBD7000L
- U$57: device vna_adapter:HEADER_3_PIN -> quadrature_generator:HEADER_3_PIN
