File: hardware/quadrature_generator.sch (EAGLE design)
At the start: 38 parts, among them IC1 74LVC1G14, IC2 74LVC74, IC3 74LVC04, IC4 74LVC04, IC5 PT7C4511, IC6 78L33

Commit message: updated component values
Parts:
- C2, C5, C7, C9: value 100n -> 1u
- C3, C4: value 1u -> 100n
- R2: value 4k7 -> 5k1
- R3: value 4k7 -> 4k3
Changed lines of the file:
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@@
 <part name="U$4" library="quadrature_generator" deviceset="GND" device=""/>
 <part name="R1" library="quadrature_generator" deviceset="R" device="1206" value="560"/>
-<part name="R2" library="quadrature_generator" deviceset="R" device="0805" value="4k7"/>
-<part name="R3" library="quadrature_generator" deviceset="R" device="0805" value="4k7"/>
+<part name="R2" library="quadrature_generator" deviceset="R" device="0805" value="5k1"/>
+<part name="R3" library="quadrature_generator" deviceset="R" device="0805" value="4k3"/>
 <part name="C1" library="quadrature_generator" deviceset="C" device="0805" value="10n"/>
 <part name="U$5" library="quadrature_generator" deviceset="GND" device=""/>
@@
 <part name="U$11" library="quadrature_generator" deviceset="+3.3V" device=""/>
 <part name="U$12" library="quadrature_generator" deviceset="GND" device=""/>
-<part name="C2" library="quadrature_generator" deviceset="C" device="0805" value="100n"/>
+<part name="C2" library="quadrature_generator" deviceset="C" device="0805" value="1u"/>
 <part name="U$13" library="quadrature_generator" deviceset="+3.3V" device=""/>
 <part name="U$14" library="quadrature_generator" deviceset="GND" device=""/>
@@
 <part name="U$19" library="quadrature_generator" deviceset="GND" device=""/>
 <part name="R4" library="quadrature_generator" deviceset="R" device="1206" value="27"/>
-<part name="C3" library="quadrature_generator" deviceset="C" device="0805" value="1u"/>
+<part name="C3" library="quadrature_generator" deviceset="C" device="0805" value="100n"/>
 <part name="U$20" library="quadrature_generator" deviceset="+3.3V" device=""/>
 <part name="U$21" library="quadrature_generator" deviceset="GND" device=""/>
@@
 <part name="U$30" library="quadrature_generator" deviceset="GND" device=""/>
 <part name="R5" library="quadrature_generator" deviceset="R" device="1206" value="27"/>
-<part name="C4" library="quadrature_generator" deviceset="C" device="0805" value="1u"/>
+<part name="C4" library="quadrature_generator" deviceset="C" device="0805" value="100n"/>
 <part name="U$3" library="quadrature_generator" deviceset="+3.3V" device=""/>
 <part name="U$8" library="quadrature_generator" deviceset="GND" device=""/>
-<part name="C5" library="quadrature_generator" deviceset="C" device="0805" value="100n"/>
+<part name="C5" library="quadrature_generator" deviceset="C" device="0805" value="1u"/>
 <part name="U$10" library="quadrature_generator" deviceset="+3.3V" device=""/>
 <part name="U$15" library="quadrature_generator" deviceset="GND" device=""/>
@@
 <part name="U$42" library="quadrature_generator" deviceset="SOLDER_BRIDGE" device=""/>
 <part name="U$43" library="quadrature_generator" deviceset="SOLDER_BRIDGE" device=""/>
-<part name="C7" library="quadrature_generator" deviceset="C" device="0805" value="100n"/>
+<part name="C7" library="quadrature_generator" deviceset="C" device="0805" value="1u"/>
 <part name="U$44" library="quadrature_generator" deviceset="+3.3V" device=""/>
 <part name="U$45" library="quadrature_generator" deviceset="GND" device=""/>
@@
 <part name="U$46" library="quadrature_generator" deviceset="GND" device=""/>
 <part name="C8" library="quadrature_generator" deviceset="C" device="0805" value="1u"/>
-<part name="C9" library="quadrature_generator" deviceset="C" device="0805" value="100n"/>
+<part name="C9" library="quadrature_generator" deviceset="C" device="0805" value="1u"/>
 <part name="U$47" library="quadrature_generator" deviceset="GND" device=""/>
 <part name="U$48" library="quadrature_generator" deviceset="GND" device=""/>
